File: v2.brd (EAGLE design)
At the start: 110.4 x 102.4 mm, 95 parts, among them IC1 ATMEGA328V-10P, IC2 LM1117DTX-3.3, J1 DCJ0202, K1 G5L, K2 G5L, K3 G5L, K4 G5L

Commit message: initial 2
Parts:
- added D11: 3mm, SparkFun-LED:FKIT-LED-1206
- added LOCK: MKDSN1,5/2-5,08, con-phoenix-508:MKDSN1,5/2-5,08
- added PWR-5, R23: 1k, resistor:M1206
- added VT5: MMBT3904LT1, transistor-npn:SOT23-BEC
Connections:
- new net DOOR1: LOCK.2, PWR-5.2, VT5.C
- new net LOCK-SIGNAL: IC1.26, R23.1
- new net N$44: D11.C, PWR-5.1
- new net N$45: R23.2, VT5.B
- net 12V0: now also LOCK.1
- net 5V0: now also D11.A
- net GND: now also VT5.E
Changed lines of the file:
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@@
 <attribute name="VALUE" x="29.46" y="76.47" size="1.27" layer="27" rot="R270"/>
+</element>
+<element name="VT5" library="transistor-npn" package="SOT23-BEC" value="MMBT3904LT1" x="2" y="-6" smashed="yes">
+<attribute name="NAME" x="3.27" y="-4.73" size="1.016" layer="25" ratio="18"/>
+<attribute name="VALUE" x="0.095" y="-9.175" size="0.8128" layer="27" ratio="10"/>
+</element>
+<element name="LOCK" library="con-phoenix-508" library_urn="urn:adsk.eagle:library:176" package="MKDSN1,5/2-5,08" package3d_urn="urn:adsk.eagle:package:9630/1" value="MKDSN1,5/2-5,08" x="5.2" y="-21.2" smashed="yes">
+<attribute name="NAME" x="0.4489" y="-16.755" size="1.27" layer="25"/>
+<attribute name="VALUE" x="12.185" y="-25.01" size="1.27" layer="27" rot="R90"/>
+</element>
+<element name="D11" library="SparkFun-LED" library_urn="urn:adsk.eagle:library:529" package="FKIT-LED-1206" package3d_urn="urn:adsk.eagle:package:39355/1" value="3mm" x="2" y="-34" smashed="yes">
+<attribute name="NAME" x="2" y="-32.88875" size="0.6096" layer="25" font="vector" ratio="20" align="bottom-center"/>
+<attribute name="VALUE" x="2" y="-35.11125" size="0.6096" layer="27" font="vector" ratio="20" align="top-center"/>
+</element>
+<element name="PWR-5" library="resistor" library_urn="urn:adsk.eagle:library:348" package="M1206" package3d_urn="urn:adsk.eagle:package:23566/1" value="1k" x="2" y="-28.8" smashed="yes">
+<attribute name="NAME" x="0.73" y="-27.53" size="1.27" layer="25"/>
+<attribute name="PWR-2" value="PWR-2" x="2" y="-32.8" size="1.778" layer="27" display="off"/>
+<attribute name="VALUE" x="0.73" y="-31.34" size="1.27" layer="27"/>
+</element>
+<element name="R23" library="resistor" library_urn="urn:adsk.eagle:library:348" package="M1206" package3d_urn="urn:adsk.eagle:package:23566/1" value="1k" x="2" y="-39.2" smashed="yes">
+<attribute name="NAME" x="0.73" y="-37.93" size="1.27" layer="25"/>
+<attribute name="VALUE" x="0.73" y="-41.74" size="1.27" layer="27"/>
 </element>
 </elements>
@@
 <wire x1="99.68" y1="23.43" x2="98.48" y2="24.63" width="1.27" layer="16"/>
 <wire x1="99.68" y1="23.43" x2="99.68" y2="18.88" width="1.27" layer="16"/>
+<contactref element="LOCK" pad="1"/>
+<wire x1="2.6389" y1="-21.175" x2="81.69" y2="18.76" width="0" layer="19" extent="1-1"/>
 </signal>
 <signal name="GND">
@@
 <contactref element="D10" pad="5"/>
 <via x="34.4" y="82.8" extent="1-16" drill="0.35"/>
+<contactref element="VT5" pad="E"/>
+<wire x1="102" y1="83.2" x2="104.4" y2="95.2" width="0" layer="19" extent="1-1"/>
+<wire x1="92.222" y1="83.999996875" x2="102" y2="83.2" width="0" layer="19" extent="1-1"/>
+<wire x1="92.222" y1="81.6" x2="92.222" y2="83.999996875" width="0" layer="19" extent="1-1"/>
+<wire x1="91.43" y1="72.77" x2="92.222" y2="81.6" width="0" layer="19" extent="1-1"/>
+<wire x1="86.63" y1="64.94" x2="91.43" y2="72.77" width="0" layer="19" extent="1-1"/>
+<wire x1="76.8" y1="69.6" x2="86.63" y2="64.94" width="0" layer="19" extent="1-1"/>
+<wire x1="68.75" y1="68.29" x2="76.8" y2="69.6" width="0" layer="19" extent="1-1"/>
+<wire x1="62.1" y1="73.56" x2="68.75" y2="68.29" width="0" layer="19" extent="1-1"/>
+<wire x1="91.83" y1="55.11" x2="86.63" y2="64.94" width="0" layer="19" extent="1-1"/>
+<wire x1="86.63" y1="46.48" x2="91.83" y2="55.11" width="0" layer="19" extent="1-1"/>
+<wire x1="87.87" y1="33.79" x2="86.63" y2="46.48" width="0" layer="19" extent="1-1"/>
+<wire x1="93.288" y1="31.96" x2="87.87" y2="33.79" width="0" layer="19" extent="1-1"/>
+<wire x1="81.16" y1="34.19" x2="87.87" y2="33.79" width="0" layer="19" extent="1-1"/>
+<wire x1="95.94" y1="24.63" x2="93.288" y2="31.96" width="0" layer="19" extent="1-1"/>
+<wire x1="96" y1="20.184" x2="95.94" y2="24.63" width="0" layer="19" extent="1-1"/>
+<wire x1="92.49" y1="15.39" x2="96" y2="20.184" width="0" layer="19" extent="1-1"/>
+<wire x1="83.82" y1="15.41" x2="92.49" y2="15.39" width="0" layer="19" extent="1-1"/>
+<wire x1="84.84" y1="21.168" x2="83.82" y2="15.41" width="0" layer="19" extent="1-1"/>
+<wire x1="77.13" y1="18.76" x2="83.82" y2="15.41" width="0" layer="19" extent="1-1"/>
+<wire x1="99.2" y1="8.8" x2="92.49" y2="15.39" width="0" layer="19" extent="1-1"/>
+<wire x1="105.42" y1="5.77" x2="99.2" y2="8.8" width="0" layer="19" extent="1-1"/>
+<wire x1="76.4" y1="7.2" x2="83.82" y2="15.41" width="0" layer="19" extent="1-1"/>
+<wire x1="72" y1="3.6" x2="76.4" y2="7.2" width="0" layer="19" extent="1-1"/>
+<wire x1="46.82" y1="71.93" x2="62.1" y2="73.56" width="0" layer="19" extent="1-1"/>
+<wire x1="46.82" y1="82.09" x2="46.82" y2="71.93" width="0" layer="19" extent="1-1"/>
+<wire x1="48.8" y1="91.2" x2="46.82" y2="82.09" width="0" layer="19" extent="1-1"/>
+<wire x1="48.8" y1="94.8" x2="48.8" y2="91.2" width="0" layer="19" extent="1-1"/>
+<wire x1="58.6" y1="97.64" x2="48.8" y2="94.8" width="0" layer="19" extent="1-1"/>
+<wire x1="68.52" y1="96.59" x2="58.6" y2="97.64" width="0" layer="19" extent="1-1"/>
+<wire x1="71.06" y1="96.59" x2="68.52" y2="96.59" width="0" layer="19" extent="1-1"/>
+<wire x1="34.4" y1="82.8" x2="46.82" y2="82.09" width="0" layer="19" extent="1-1"/>
+<wire x1="30.1" y1="82.8" x2="34.4" y2="82.8" width="0" layer="19" extent="1-1"/>
+<wire x1="28.4" y1="82.8" x2="30.1" y2="82.8" width="0" layer="19" extent="1-1"/>
+<wire x1="26.7" y1="82.8" x2="28.4" y2="82.8" width="0" layer="19" extent="1-1"/>
+<wire x1="31.23" y1="93.29" x2="30.1" y2="82.8" width="0" layer="19" extent="1-1"/>
+<wire x1="35.92" y1="60.84" x2="46.82" y2="71.93" width="0" layer="19" extent="1-1"/>
+<wire x1="25.78" y1="57.64" x2="35.92" y2="60.84" width="0" layer="19" extent="1-1"/>
+<wire x1="25.9" y1="54.84" x2="25.78" y2="57.64" width="0" layer="19" extent="1-1"/>
+<wire x1="21.2" y1="49.01" x2="25.9" y2="54.84" width="0" layer="19" extent="1-1"/>
+<wire x1="38.4" y1="49.01" x2="35.92" y2="60.84" width="0" layer="19" extent="1-1"/>
+<wire x1="11.56" y1="63.872" x2="25.78" y2="57.64" width="0" layer="19" extent="1-1"/>
+<wire x1="11.56" y1="73.148" x2="11.56" y2="63.872" width="0" layer="19" extent="1-1"/>
+<wire x1="4.425" y1="71.8811" x2="11.56" y2="73.148" width="0" layer="19" extent="1-1"/>
+<wire x1="5.64" y1="48.8" x2="21.2" y2="49.01" width="0" layer="19" extent="1-1"/>
+<wire x1="12.36" y1="35.2" x2="5.64" y2="48.8" width="0" layer="19" extent="1-1"/>
+<wire x1="13.6" y1="33.6" x2="12.36" y2="35.2" width="0" layer="19" extent="1-1"/>
+<wire x1="28.76" y1="35.29" x2="13.6" y2="33.6" width="0" layer="19" extent="1-1"/>
+<wire x1="45.96" y1="35.38" x2="38.4" y2="49.01" width="0" layer="19" extent="1-1"/>
+<wire x1="60.8" y1="35.2" x2="45.96" y2="35.38" width="0" layer="19" extent="1-1"/>
+<wire x1="63.16" y1="35.07" x2="60.8" y2="35.2" width="0" layer="19" extent="1-1"/>
+<wire x1="54.4" y1="49.01" x2="60.8" y2="35.2" width="0" layer="19" extent="1-1"/>
+<wire x1="53.6" y1="53.2" x2="54.4" y2="49.01" width="0" layer="19" extent="1-1"/>
+<wire x1="13.74" y1="93.29" x2="26.7" y2="82.8" width="0" layer="19" extent="1-1"/>
+<wire x1="4.96" y1="93.61" x2="13.74" y2="93.29" width="0" layer="19" extent="1-1"/>
+<wire x1="4.47" y1="4.41" x2="13.6" y2="33.6" width="0" layer="19" extent="1-1"/>
+<wire x1="2.95" y1="-7.1" x2="4.47" y2="4.41" width="0" layer="19" extent="1-1"/>
 </signal>
 <signal name="5V0">
@@
 <wire x1="4.4" y1="42.4" x2="5.6" y2="42.4" width="0.4064" layer="16"/>
 <wire x1="5.6" y1="42.4" x2="5.64" y2="41.18" width="0.4064" layer="16"/>
+<contactref element="D11" pad="A"/>
+<wire x1="5.6" y1="22.4" x2="0.578" y2="-34" width="0" layer="19" extent="1-1"/>
 </signal>
 <signal name="N$25">
@@
 <wire x1="28.4" y1="75.022" x2="28.4" y2="78" width="0.4064" layer="1"/>
 </signal>
+<signal name="DOOR1">
+<contactref element="LOCK" pad="2"/>
+<contactref element="VT5" pad="C"/>
+<contactref element="PWR-5" pad="2"/>
+<wire x1="7.7189" y1="-21.175" x2="3.4" y2="-28.8" width="0" layer="19" extent="1-1"/>
+<wire x1="2" y1="-4.9" x2="7.7189" y2="-21.175" width="0" layer="19" extent="1-1"/>
+</signal>
+<signal name="N$44">
+<contactref element="D11" pad="C"/>
+<contactref element="PWR-5" pad="1"/>
+<wire x1="0.6" y1="-28.8" x2="3.422" y2="-34" width="0" layer="19" extent="1-1"/>
+</signal>
+<signal name="N$45">
+<contactref element="VT5" pad="B"/>
+<contactref element="R23" pad="2"/>
+<wire x1="1.05" y1="-7.1" x2="3.4" y2="-39.2" width="0" layer="19" extent="1-1"/>
+</signal>
+<signal name="LOCK-SIGNAL">
+<contactref element="R23" pad="1"/>
+<contactref element="IC1" pad="26"/>
+<wire x1="0.6" y1="-39.2" x2="23.22" y2="68.46" width="0" layer="19" extent="1-1"/>
+</signal>
 </signals>
